File: hardware/novapad/NovaPad.kicad_pcb (KiCad board)
At the start: 2 copper layers, 74 x 50 mm, 4 parts, among them J1 GND SW1 SW2 SW3, SW1 SW_Tactile_6mm, SW2 SW_Tactile_6mm, SW3 SW_Tactile_6mm

Commit message: Complete three-button PCB wiring
Co-authored-by: bminsky35 <95700515+bminsky35@users.noreply.github.com>
Routing:
- added copper zone on B.Cu, net GND
Changed lines of the file:
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@@
 (kicad_pcb
-  (version 20241229)
+  (version 20221018)
   (generator "pcbnew")
   (general
@@
   (net 3 "SW2")
   (net 4 "SW3")
+  (zone
+    (net 1)
+    (net_name "GND")
+    (layer "B.Cu")
+    (hatch edge 0.5)
+    (connect_pads (clearance 0.2))
+    (min_thickness 0.25)
+    (fill yes (thermal_gap 0.3) (thermal_bridge_width 0.3))
+    (polygon
+      (pts
+        (xy 4 4)
+        (xy 76 4)
+        (xy 76 52)
+        (xy 4 52)
+      )
+    )
+  )
   (gr_rect
     (start 3 3)
@@
   )
   (footprint "NovaPad:SW_Tactile_6mm" (layer "F.Cu") (at 16 18)
-    (property "Reference" "SW1" (at 0 -6) (layer "F.SilkS")
+    (property "Reference" "SW1" (at 16 12) (layer "F.SilkS")
       (effects (font (size 1 1) (thickness 0.15)))
     )
-    (property "Value" "SW_Tactile_6mm" (at 0 6) (layer "F.Fab")
+    (property "Value" "SW_Tactile_6mm" (at 16 24) (layer "F.Fab")
       (effects (font (size 0.8 0.8) (thickness 0.12)))
     )
@@
   )
   (footprint "NovaPad:SW_Tactile_6mm" (layer "F.Cu") (at 40 18)
-    (property "Reference" "SW2" (at 0 -6) (layer "F.SilkS")
+    (property "Reference" "SW2" (at 40 12) (layer "F.SilkS")
       (effects (font (size 1 1) (thickness 0.15)))
     )
-    (property "Value" "SW_Tactile_6mm" (at 0 6) (layer "F.Fab")
+    (property "Value" "SW_Tactile_6mm" (at 40 24) (layer "F.Fab")
       (effects (font (size 0.8 0.8) (thickness 0.12)))
     )
@@
   )
   (footprint "NovaPad:SW_Tactile_6mm" (layer "F.Cu") (at 64 18)
-    (property "Reference" "SW3" (at 0 -6) (layer "F.SilkS")
+    (property "Reference" "SW3" (at 64 12) (layer "F.SilkS")
       (effects (font (size 1 1) (thickness 0.15)))
     )
-    (property "Value" "SW_Tactile_6mm" (at 0 6) (layer "F.Fab")
+    (property "Value" "SW_Tactile_6mm" (at 64 24) (layer "F.Fab")
       (effects (font (size 0.8 0.8) (thickness 0.12)))
     )
@@
   )
   (footprint "NovaPad:PinHeader_1x04_P2.54mm" (layer "F.Cu") (at 40 44.2)
-    (property "Reference" "J1" (at 3.5 -3.5) (layer "F.SilkS")
+    (property "Reference" "J1" (at 43.5 40.7) (layer "F.SilkS")
       (effects (font (size 1 1) (thickness 0.15)))
     )
-    (property "Value" "GND SW1 SW2 SW3" (at 3.5 3.5) (layer "F.Fab")
+    (property "Value" "GND SW1 SW2 SW3" (at 43.5 47.7) (layer "F.Fab")
       (effects (font (size 0.8 0.8) (thickness 0.12)))
     )
